Commit message: Adding pattern and making simulation work

File: softbot2_description/urdf/open_manipulator_x.gazebo.xacro (robot description, xacro)
@@ -10,5 +10,5 @@
       <maxVel>1.0</maxVel>
       <minDepth>0.001</minDepth>
-      <material>Gazebo/DarkGrey</material>
+      <material>Gazebo/Orange</material>
     </gazebo>
   </xacro:macro>

File: softbot2_description/urdf/open_manipulator_x.urdf.xacro (robot description, xacro)
@@ -5,4 +5,7 @@
   <!-- Include OpenManipulator Transmission -->
   <xacro:include filename="$(find turtlebot3_manipulation_description)/urdf/open_manipulator_x.transmission.xacro"/>
+  <material name="light_grey">
+    <color rgba="0.7 0.7 0.7 1.0"/>
+  </material>
   <!-- Link 1 -->
   <link name="link1">
@@ -12,5 +15,5 @@
         <mesh filename="package://turtlebot3_manipulation_description/meshes/chain_link1.stl" scale="0.001 0.001 0.001"/>
       </geometry>
-      <material name="grey"/>
+      <material name="light_grey"/>
     </visual>
     <collision>
@@ -43,5 +46,6 @@
         <mesh filename="package://turtlebot3_manipulation_description/meshes/chain_link2.stl" scale="0.001 0.001 0.001"/>
       </geometry>
-      <material name="grey"/>
+      <!-- <material name="grey"/> -->
+      <material name="light_grey"/>
     </visual>
     <collision>
@@ -74,5 +78,6 @@
         <mesh filename="package://turtlebot3_manipulation_description/meshes/chain_link3.stl" scale="0.001 0.001 0.001"/>
       </geometry>
-      <material name="grey"/>
+      <material name="light_grey"/>
+      <!-- <material name="grey"/> -->
     </visual>
     <collision>
@@ -105,5 +110,6 @@
         <mesh filename="package://turtlebot3_manipulation_description/meshes/chain_link4.stl" scale="0.001 0.001 0.001"/>
       </geometry>
-      <material name="grey"/>
+      <!-- <material name="grey"/> -->
+      <material name="light_grey"/>
     </visual>
     <collision>
@@ -136,5 +142,6 @@
         <mesh filename="package://turtlebot3_manipulation_description/meshes/chain_link5.stl" scale="0.001 0.001 0.001"/>
       </geometry>
-      <material name="grey"/>
+      <!-- <material name="grey"/> -->
+      <material name="light_grey"/>
     </visual>
     <collision>
@@ -163,5 +170,6 @@
         <mesh filename="package://turtlebot3_manipulation_description/meshes/chain_link_grip_l.stl" scale="0.001 0.001 0.001"/>
       </geometry>
-      <material name="grey"/>
+      <material name="light_grey"/>
+      <!-- <material name="grey"/> -->
     </visual>
     <collision>
@@ -194,5 +202,6 @@
         <mesh filename="package://turtlebot3_manipulation_description/meshes/chain_link_grip_r.stl" scale="0.001 0.001 0.001"/>
       </geometry>
-      <material name="grey"/>
+      <!-- <material name="grey"/> -->
+      <material name="light_grey"/>
     </visual>
     <collision>
@@ -230,7 +239,8 @@
       <origin xyz="0 0 0" rpy="0 0 0"/>
       <geometry>
-        <box size="0.01 0.01 0.01" />
-      </geometry>
-      <material name="red"/>
+        <box size="0.001 0.001 0.001" />
+      </geometry>
+      <!-- <material name="red"/> -->
+      <material name="light_grey"/>
      </visual>
     <inertial>

File: softbot2_description/urdf/softbot2.urdf.xacro (robot description, xacro)
@@ -72,8 +72,8 @@
     <inertial>
       <origin xyz="0 0 0" />
-      <mass value="2.8498940e-02" />
-      <inertia ixx="1.1175580e-05" ixy="-4.2369783e-11" ixz="-5.9381719e-09"
-               iyy="1.1192413e-05" iyz="-1.4400107e-11"
-               izz="2.0712558e-05" />
+      <mass value="2.8498940e-01" />
+      <inertia ixx="1.1175580e-03" ixy="-4.2369783e-11" ixz="-5.9381719e-09"
+               iyy="1.1192413e-03" iyz="-1.4400107e-11"
+               izz="2.0712558e-03" />
     </inertial>
   </link>
@@ -100,8 +100,8 @@
     <inertial>
       <origin xyz="0 0 0" />
-      <mass value="2.8498940e-02" />
-      <inertia ixx="1.1175580e-05" ixy="-4.2369783e-11" ixz="-5.9381719e-09"
-               iyy="1.1192413e-05" iyz="-1.4400107e-11"
-               izz="2.0712558e-05" />
+      <mass value="2.8498940e-01" />
+      <inertia ixx="1.1175580e-03" ixy="-4.2369783e-11" ixz="-5.9381719e-09"
+               iyy="1.1192413e-03" iyz="-1.4400107e-11"
+               izz="2.0712558e-03" />
     </inertial>
   </link>
@@ -225,22 +225,22 @@
     <origin xyz="0 0 0" rpy="0 0 0" />
   </xacro:VLP-16_blue>
-  <link name="front_left_camera_support_link">
-  </link>
-  <joint name="platform_support_leg3_link_to_front_left_camera_support_link" type="fixed">
-    <origin xyz="0.02 0 -0.09" rpy="0.01 -0.35 0.2"/>
+  <link name="body_camera_support_link">
+  </link>
+  <joint name="platform_support_leg3_link_to_body_camera_support_link" type="fixed">
+    <origin xyz="0.02 -0.05 -0.13" rpy="0.01 -0.35 0.05"/>
     <parent link="platform_support_leg3_link"/>
-    <child link="front_left_camera_support_link"/>
-  </joint>
-  <xacro:sensor_astra_red prefix="front_left_camera" parent="front_left_camera_support_link">
+    <child link="body_camera_support_link"/>
+  </joint>
+  <xacro:sensor_astra_red prefix="body_camera" parent="body_camera_support_link">
     <origin xyz="0.02 0.07 0.015" rpy="0 0.0 0" />
   </xacro:sensor_astra_red>
-  <link name="front_right_camera_support_link">
-  </link>
-  <joint name="platform_support_leg4_link_to_front_right_camera_support_link" type="fixed">
-    <origin xyz="0.02 0 -0.05" rpy="0.01 -0.35 -0.22"/>
-    <parent link="platform_support_leg4_link"/>
-    <child link="front_right_camera_support_link"/>
-  </joint>
-  <xacro:sensor_astra_green prefix="front_right_camera" parent="front_right_camera_support_link">
+  <link name="hand_camera_support_link">
+  </link>
+  <joint name="end_effector_link_to_hand_camera_support_link" type="fixed">
+    <origin xyz="-0.08 0 0.04" rpy="0.0 0.0 0.0"/>
+    <parent link="end_effector_link"/>
+    <child link="hand_camera_support_link"/>
+  </joint>
+  <xacro:sensor_astra_green prefix="hand_camera" parent="hand_camera_support_link">
     <origin xyz="0.02 0.07 0.015" rpy="0 0.0 0" />
   </xacro:sensor_astra_green>
